Commit message: IMU frame added

File: urdf/my_robot.urdf (robot description, URDF)
Before this commit: robot robot_wheeled, 5 links, 4 joints
Links:
- added link imu, mass 0.05
- link robot_base_link: geometry collision box size=2.0 1.0 0.46; visual box size=2.0 1.0 0.5
Joints:
- added joint imu_joint: type fixed, parent robot_base_link, child imu, origin xyz=0 0 0.45 rpy=0 0 0
- joint caster_wheel: origin xyz=0.8 0 -0.2 rpy=0 0 0 -> xyz=0.8 0 0.2 rpy=0 0 0
- joint left_wheel_joint: origin xyz=-0.5 0.6 0 rpy=-1.5707 0 0 -> xyz=-0.5 0.6 0.4 rpy=-1.5707 0 0
- joint lidar_joint: origin xyz=0.8 0 0.5 rpy=0 0 0 -> xyz=0.8 0 0.76 rpy=0 0 0
- joint right_wheel_joint: origin xyz=-0.5 -0.6 0 rpy=-1.5707 0 0 -> xyz=-0.5 -0.6 0.4 rpy=-1.5707 0 0
