Commit message: fix: urdf for gz harmonic

File: evarobot_description/urdf/evarobot.gazebo.xacro (robot description, xacro)
@@ -1,9 +1,11 @@
 <?xml version="1.0"?>
 <!--
-  EvaRobot Gazebo Configuration
-  Gazebo-specific elements including:
+  EvaRobot Gazebo Harmonic Configuration
+  Gazebo Harmonic-specific elements including:
   - Material colors
   - Physical properties (friction, damping)
-  - Sensor plugins (if needed)
+  - Sensor plugins (IMU, LiDAR)
+  Note: This file is configured for Gazebo Harmonic (gz-sim) used with ROS2 Jazzy.
+        For Gazebo Classic, use different plugin names.
   Author: Kevin Medrano Ayala
   License: BSD-3-Clause
@@ -11,5 +13,5 @@
 <robot xmlns:xacro="http://www.ros.org/wiki/xacro">
   <!-- ===================================================================== -->
-  <!-- GAZEBO COLORS -->
+  <!-- GAZEBO COLORS AND PHYSICS -->
   <!-- ===================================================================== -->
   <gazebo reference="base_link">
@@ -46,7 +48,11 @@
   </gazebo>
   <!-- ===================================================================== -->
-  <!-- ADDITIONAL SENSORS (OPTIONAL) -->
+  <!-- GAZEBO HARMONIC SENSORS (OPTIONAL) -->
   <!-- ===================================================================== -->
-  <!-- Example: IMU sensor (commented out, add if needed) -->
+  <!--
+    IMU Sensor for Gazebo Harmonic
+    Uncomment to enable IMU sensor on the robot.
+    Note: Requires 'imu_link' to be defined in the URDF.
+  -->
   <!--
   <gazebo reference="base_link">
@@ -54,26 +60,25 @@
       <always_on>true</always_on>
       <update_rate>100</update_rate>
-      <plugin name="imu_plugin" filename="libgazebo_ros_imu_sensor.so">
-        <ros>
-          <namespace>/</namespace>
-          <remapping>~/out:=imu</remapping>
-        </ros>
-        <initial_orientation_as_reference>false</initial_orientation_as_reference>
-      </plugin>
+      <topic>imu</topic>
+      <gz_frame_id>base_link</gz_frame_id>
+      <enable_metrics>false</enable_metrics>
     </sensor>
   </gazebo>
   -->
-  <!-- Example: Lidar sensor (commented out, add if needed) -->
+  <!--
+    LiDAR Sensor for Gazebo Harmonic
+    Uncomment to enable LiDAR sensor on the robot.
+    Note: Requires 'lidar_link' to be defined in the URDF.
+  -->
   <!--
   <gazebo reference="base_link">
-    <sensor name="lidar" type="ray">
-      <always_on>true</always_on>
-      <visualize>true</visualize>
+    <sensor name="lidar" type="gpu_lidar">
+      <topic>scan</topic>
       <update_rate>10</update_rate>
-      <ray>
+      <lidar>
         <scan>
           <horizontal>
             <samples>360</samples>
-            <resolution>1.0</resolution>
+            <resolution>1</resolution>
             <min_angle>-3.14159</min_angle>
             <max_angle>3.14159</max_angle>
@@ -90,13 +95,39 @@
           <stddev>0.01</stddev>
         </noise>
-      </ray>
-      <plugin name="scan" filename="libgazebo_ros_ray_sensor.so">
-        <ros>
-          <namespace>/</namespace>
-          <remapping>~/out:=scan</remapping>
-        </ros>
-        <output_type>sensor_msgs/LaserScan</output_type>
-        <frame_name>lidar_link</frame_name>
-      </plugin>
+      </lidar>
+      <always_on>true</always_on>
+      <visualize>true</visualize>
+    </sensor>
+  </gazebo>
+  -->
+  <!--
+    Camera Sensor for Gazebo Harmonic
+    Uncomment to enable camera sensor on the robot.
+    Note: Requires 'camera_link' to be defined in the URDF.
+  -->
+  <!--
+  <gazebo reference="base_link">
+    <sensor name="camera" type="camera">
+      <topic>camera</topic>
+      <update_rate>30</update_rate>
+      <camera>
+        <horizontal_fov>1.047</horizontal_fov>
+        <image>
+          <width>640</width>
+          <height>480</height>
+          <format>R8G8B8</format>
+        </image>
+        <clip>
+          <near>0.1</near>
+          <far>100</far>
+        </clip>
+        <noise>
+          <type>gaussian</type>
+          <mean>0.0</mean>
+          <stddev>0.007</stddev>
+        </noise>
+      </camera>
+      <always_on>true</always_on>
+      <visualize>true</visualize>
     </sensor>
   </gazebo>

File: evarobot_description/urdf/evarobot.ros2_control.xacro (robot description, xacro)
@@ -3,6 +3,6 @@
   EvaRobot ROS2 Control Configuration
   Defines the hardware interface for ROS2 Control.
-  For Gazebo simulation, uses gazebo_ros2_control plugin.
-  For real hardware, this would be replaced with custom hardware interface.
+  Configured for Gazebo Harmonic simulation using gz_ros2_control plugin.
+  For real hardware, replace the hardware plugin with your custom hardware interface.
   Author: Kevin Medrano Ayala
   License: BSD-3-Clause
@@ -13,7 +13,5 @@
   <!-- ===================================================================== -->
   <ros2_control name="evarobot_system" type="system">
-    <!-- Hardware plugin -->
-    <!-- For Gazebo Harmonic simulation, use gz_ros2_control/GazeboSimSystem -->
-    <!-- For Gazebo Classic, use: gazebo_ros2_control/GazeboSystem -->
+    <!-- Hardware plugin for Gazebo Harmonic simulation -->
     <!-- For real hardware, replace with your custom hardware interface -->
     <hardware>
@@ -40,8 +38,8 @@
   </ros2_control>
   <!-- ===================================================================== -->
-  <!-- GAZEBO ROS2 CONTROL PLUGIN -->
+  <!-- GAZEBO HARMONIC ROS2 CONTROL PLUGIN -->
   <!-- ===================================================================== -->
   <gazebo>
-    <!-- For Gazebo Harmonic (ROS2 Jazzy) -->
+    <!-- Gazebo Harmonic ROS2 Control Plugin -->
     <plugin filename="libgz_ros2_control-system.so" name="gz_ros2_control::GazeboSimROS2ControlPlugin">
       <!-- ROS2 Control configuration file -->
@@ -52,12 +50,4 @@
       </ros>
     </plugin>
-    <!-- For Gazebo Classic (ROS2 Humble and earlier), use this instead:
-    <plugin filename="libgazebo_ros2_control.so" name="gazebo_ros2_control">
-      <parameters>$(find evarobot_controller)/config/evarobot_controllers.yaml</parameters>
-      <ros>
-        <namespace>/</namespace>
-      </ros>
-    </plugin>
-    -->
   </gazebo>
 </robot>

File: evarobot_description/urdf/evarobot.urdf.xacro (robot description, xacro)
@@ -17,6 +17,6 @@
   <!-- Robot dimensions (meters) -->
   <xacro:property name="base_length" value="0.30" />
-  <xacro:property name="base_width" value="0.20" />
-  <xacro:property name="base_height" value="0.08" />
+  <xacro:property name="base_width" value="0.16" />  <!-- Reduced from 0.20 so wheels stick out -->
+  <xacro:property name="base_height" value="0.056" />  <!-- Reduced by 30% from 0.08 to show wheels better -->
   <xacro:property name="base_mass" value="2.0" />
   <!-- Wheel dimensions (measured from evarobot_controllers.yaml) -->
