Commit message: Reposition driven wheels 30% backwards from center
- Add wheel_offset_x property (-0.09m, 30% of base_length)
- Move driven wheels from center (x=0) to back (x=-0.09m)
- Caster wheel remains at front (x=+0.12m)
- Improves stability and control for differential drive

Classic configuration: caster front, driven wheels back.

🤖 Generated with [Claude Code](https://claude.com/claude-code)

Co-Authored-By: Claude <noreply@anthropic.com>

File: evarobot_description/urdf/evarobot.urdf.xacro (robot description, xacro)
@@ -25,4 +25,6 @@
   <xacro:property name="wheel_mass" value="0.1" />
   <xacro:property name="wheel_separation" value="0.194" />
+  <!-- Wheel position offset (30% of base_length backwards from center) -->
+  <xacro:property name="wheel_offset_x" value="${-0.3 * base_length}" />
   <!-- Caster wheel dimensions -->
   <xacro:property name="caster_radius" value="0.015" />
@@ -118,5 +120,5 @@
       <parent link="base_link"/>
       <child link="${prefix}_wheel_link"/>
-      <origin xyz="0 ${reflect * wheel_separation / 2.0} 0" rpy="0 0 0"/>
+      <origin xyz="${wheel_offset_x} ${reflect * wheel_separation / 2.0} 0" rpy="0 0 0"/>
       <axis xyz="0 1 0"/>
     </joint>
